File: hw/flashrom.kicad_pcb (KiCad board)
At the start: 2 copper layers, 18.3 x 52.1 mm, 14 parts, among them J1 Conn_01x04_Pin, J2 Conn_01x03_Pin, J3 Conn_01x04_Pin, U1 29F800-TSOP, U2 Kickstart_Socket_A4000

Commit message: increase pull-ups to 18k, the value actually used in the protos
Parts:
- R3, R4, R5, R6, R7: value 15k -> 18k
Changed lines of the file:
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@@
     (property "Sheetfile" "flashrom.kicad_sch")
     (property "Sheetname" "")
-    (property "dnp" "")
-    (property "exclude_from_bom" "")
-    (property "ki_description" "Resistor, small symbol")
-    (property "ki_keywords" "R resistor")
-    (attr smd exclude_from_bom)
+    (property "ki_description" "Resistor, small symbol")
+    (property "ki_keywords" "R resistor")
+    (attr smd)
     (fp_text reference "R7" (at -2.985 0 90 unlocked) (layer "B.SilkS")
         (effects (font (size 1 0.8) (thickness 0.12)) (justify mirror))
     )
-    (fp_text value "15k" (at 0 -1.43 90) (layer "B.Fab")
+    (fp_text value "18k" (at 0 -1.43 90) (layer "B.Fab")
         (effects (font (size 1 1) (thickness 0.15)) (justify mirror))
     )
@@
         (effects (font (size 1 0.8) (thickness 0.12)) (justify mirror))
     )
-    (fp_text value "15k" (at 0 -1.43 90) (layer "B.Fab")
+    (fp_text value "18k" (at 0 -1.43 90) (layer "B.Fab")
         (effects (font (size 1 1) (thickness 0.15)) (justify mirror))
     )
@@
         (effects (font (size 1 0.8) (thickness 0.12)) (justify mirror))
     )
-    (fp_text value "15k" (at 0 -1.43 90) (layer "B.Fab")
+    (fp_text value "18k" (at 0 -1.43 90) (layer "B.Fab")
         (effects (font (size 1 1) (thickness 0.15)) (justify mirror))
     )
@@
         (effects (font (size 1 0.8) (thickness 0.12)) (justify mirror))
     )
-    (fp_text value "15k" (at 0 -1.43 -270) (layer "B.Fab")
+    (fp_text value "18k" (at 0 -1.43 -270) (layer "B.Fab")
         (effects (font (size 1 1) (thickness 0.15)) (justify mirror))
     )
@@
         (effects (font (size 1 0.8) (thickness 0.12)) (justify mirror))
     )
-    (fp_text value "15k" (at 0 -1.43 90) (layer "B.Fab")
-        (effects (font (size 1 1) (thickness 0.15)) (justify mirror))
-    )
+    (fp_text value "18k" (at 0 -1.43 90) (layer "B.Fab")
+        (effects (font (size 1 1) (thickness 0.15)) (justify mirror))
+    )
