File: flash_adapter/flash_adapter.kicad_sch (KiCad schematic)
At the start: 5 parts, among them J1 Conn_02x12_Odd_Even, J2 Conn_02x12_Odd_Even, J4 Conn_01x04_Pin, U1 Kickstart_Socket_A4000, U2 29F800

Commit message: increase dip 40 socket hole size in order to allow use of textool socket
Parts:
- U1: footprint Package_DIP:DIP-40_W15.24mm_Socket -> Package_DIP:DIP-40_W15.24mm_Socket_LongPads
Changed lines of the file:
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@@
       (effects (font (size 1.27 1.27)))
     )
-    (property "Footprint" "Package_DIP:DIP-40_W15.24mm_Socket" (at 60.96 151.13 0)
+    (property "Footprint" "Package_DIP:DIP-40_W15.24mm_Socket_LongPads" (at 60.96 151.13 0)
       (effects (font (size 1.27 1.27)) (justify left) hide)
     )

Commit message: update schematic legend
Other:
- title: (none) -> Flash adapter for TL866
Changed lines of the file:
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@@
 (kicad_sch (version 20230121) (generator eeschema)
   (paper "A4")
+  (title_block
+    (title "Flash adapter for TL866")
+    (date "2025-01-12")
+    (rev "2")
+    (comment 1 "Original by github.com/matthiesenj")
+    (comment 2 "Requires TL866 TSOP48/SOP44 adapter")
+  )
   (no_connect (at 194.31 118.11))
   (no_connect (at 194.31 110.49))

Commit message: relocate header for non-socket signals to next to socket to avoid through holes under textool
Other:
- title: Flash adapter for TL866 -> FlashROM programming adapter for TL866
Changed lines of the file:
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@@
   (paper "A4")
   (title_block
-    (title "Flash adapter for TL866")
-    (date "2025-01-12")
-    (rev "2")
+    (title "FlashROM programming adapter for TL866")
+    (date "2025-01-26")
+    (rev "3")
     (comment 1 "Original by github.com/matthiesenj")
     (comment 2 "Requires TL866 TSOP48/SOP44 adapter")
